Commit message: simple changes

File: notspot_description/urdf/notspot.urdf.xacro (robot description, xacro)
@@ -302,5 +302,5 @@
     <axis xyz="0 0 1" />
     <limit lower="-3" upper="3" effort="${effort_limit}" velocity="3" />
-    <dynamics damping="0.7" friction="10.0" />
+    <dynamics damping="10.0" friction="1000.0" />
   </joint>
   <joint name="FR2_joint" type="revolute">
@@ -310,5 +310,5 @@
     <axis xyz="0 0 1" />
     <limit lower="-3" upper="3" effort="${effort_limit}" velocity="3" />
-    <dynamics damping="0.7" friction="10.0" />
+    <dynamics damping="10.0" friction="1000.0" />
   </joint>
   <joint name="FR3_joint" type="revolute">
@@ -318,5 +318,5 @@
     <axis xyz="0 0 1" />
     <limit lower="-3" upper="3" effort="${effort_limit}" velocity="3" />
-    <dynamics damping="0.7" friction="10.0" />
+    <dynamics damping="10.0" friction="1000.0" />
   </joint>
   <joint name="FR4_joint" type="fixed">
@@ -332,5 +332,5 @@
     <axis xyz="0 0 1" />
     <limit lower="-3" upper="3" effort="${effort_limit}" velocity="3" />
-    <dynamics damping="0.7" friction="10.0" />
+    <dynamics damping="10.0" friction="1000.0" />
   </joint>
   <joint name="FL2_joint" type="revolute">
@@ -340,5 +340,5 @@
     <axis xyz="0 0 1" />
     <limit lower="-3" upper="3" effort="${effort_limit}" velocity="3" />
-    <dynamics damping="0.7" friction="10.0" />
+    <dynamics damping="10.0" friction="1000.0" />
   </joint>
   <joint name="FL3_joint" type="revolute">
@@ -348,5 +348,5 @@
     <axis xyz="0 0 1" />
     <limit lower="-3" upper="3" effort="${effort_limit}" velocity="3" />
-    <dynamics damping="0.7" friction="10.0" />
+    <dynamics damping="10.0" friction="1000.0" />
   </joint>
   <joint name="FL4_joint" type="fixed">
@@ -362,5 +362,5 @@
     <axis xyz="0 0 1" />
     <limit lower="-3" upper="3" effort="${effort_limit}" velocity="3" />
-    <dynamics damping="0.7" friction="10.0" />
+    <dynamics damping="10.0" friction="1000.0" />
   </joint>
   <joint name="RR2_joint" type="revolute">
@@ -370,5 +370,5 @@
     <axis xyz="0 0 1" />
     <limit lower="-3" upper="3" effort="${effort_limit}" velocity="3" />
-    <dynamics damping="0.7" friction="10.0" />
+    <dynamics damping="10.0" friction="1000.0" />
   </joint>
   <joint name="RR3_joint" type="revolute">
@@ -378,5 +378,5 @@
     <axis xyz="0 0 1" />
     <limit lower="-3" upper="3" effort="${effort_limit}" velocity="3" />
-    <dynamics damping="0.7" friction="10.0" />
+    <dynamics damping="10.0" friction="1000.0" />
   </joint>
   <joint name="RR4_joint" type="fixed">
@@ -392,5 +392,5 @@
     <axis xyz="0 0 1" />
     <limit lower="-3" upper="3" effort="${effort_limit}" velocity="3" />
-    <dynamics damping="0.7" friction="10.0" />
+    <dynamics damping="10.0" friction="1000.0" />
   </joint>
   <joint name="RL2_joint" type="revolute">
@@ -400,5 +400,5 @@
     <axis xyz="0 0 1" />
     <limit lower="-3" upper="3" effort="${effort_limit}" velocity="3" />
-    <dynamics damping="0.7" friction="10.0" />
+    <dynamics damping="10.0" friction="1000.0" />
   </joint>
   <joint name="RL3_joint" type="revolute">
@@ -408,5 +408,5 @@
     <axis xyz="0 0 1" />
     <limit lower="-3" upper="3" effort="${effort_limit}" velocity="3" />
-    <dynamics damping="0.7" friction="10.0" />
+    <dynamics damping="10.0" friction="1000.0" />
   </joint>
   <joint name="RL4_joint" type="fixed">
@@ -671,33 +671,89 @@
   <!-- FR4 friction -->
   <gazebo reference="FR4">
-    <mu1>1.0</mu1>
-    <mu2>1.0</mu2>
-    <minDepth>0.0002</minDepth>
-    <kp value="1000000.0" />
-    <kd value="100.0" />
+    <collision>
+      <surface>
+        <friction>
+          <ode>
+            <mu>1</mu>
+            <mu2>100</mu2>
+            <slip1>0.0</slip1>
+            <slip2>0.0</slip2>
+          </ode>
+        </friction>
+        <contact>
+          <ode>
+            <kp>1000000.0</kp>
+            <kd>100.0</kd>
+            <min_depth>0.001</min_depth>
+          </ode>
+        </contact>
+      </surface>
+    </collision>
   </gazebo>
   <!-- FL4 friction -->
   <gazebo reference="FL4">
-    <mu1>1.0</mu1>
-    <mu2>1.0</mu2>
-    <minDepth>0.0002</minDepth>
-    <kp value="1000000.0" />
-    <kd value="100.0" />
+    <collision>
+      <surface>
+        <friction>
+          <ode>
+            <mu>1</mu>
+            <mu2>100</mu2>
+            <slip1>0.0</slip1>
+            <slip2>0.0</slip2>
+          </ode>
+        </friction>
+        <contact>
+          <ode>
+            <kp>1000000.0</kp>
+            <kd>100.0</kd>
+            <min_depth>0.001</min_depth>
+          </ode>
+        </contact>
+      </surface>
+    </collision>
   </gazebo>
   <!-- RR4 friction -->
   <gazebo reference="RR4">
-    <mu1>1.0</mu1>
-    <mu2>1.0</mu2>
-    <minDepth>0.0002</minDepth>
-    <kp value="1000000.0" />
-    <kd value="100.0" />
+    <collision>
+      <surface>
+        <friction>
+          <ode>
+            <mu>1</mu>
+            <mu2>100</mu2>
+            <slip1>0.0</slip1>
+            <slip2>0.0</slip2>
+          </ode>
+        </friction>
+        <contact>
+          <ode>
+            <kp>1000000.0</kp>
+            <kd>100.0</kd>
+            <min_depth>0.001</min_depth>
+          </ode>
+        </contact>
+      </surface>
+    </collision>
   </gazebo>
   <!-- RL4 friction -->
   <gazebo reference="RL4">
-    <mu1>1.0</mu1>
-    <mu2>1.0</mu2>
-    <minDepth>0.0002</minDepth>
-    <kp value="1000000.0" />
-    <kd value="100.0" />
+    <collision>
+      <surface>
+        <friction>
+          <ode>
+            <mu>1</mu>
+            <mu2>100</mu2>
+            <slip1>100.1</slip1>
+            <slip2>100.1</slip2>
+          </ode>
+        </friction>
+        <contact>
+          <ode>
+            <kp>1000000.0</kp>
+            <kd>100.0</kd>
+            <min_depth>0.001</min_depth>
+          </ode>
+        </contact>
+      </surface>
+    </collision>
   </gazebo>
 </robot>
